File: vaucasy_right/vaucasy_right.kicad_sch (KiCad schematic)
At the start: 105 parts, among them J1 USB_C, J2 OLED_128x32, J4 Trackball, J5 HC-05 BT, J6 DEBUG, SW1 SW_SPDT, SW2 SW_Push, SW3 RotaryEncoder_Switch, U1 STM32F401RET6, U2 USBLC6-2SC6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

Commit message: ordered
Parts:
- added H1, H2, H3: MountingHole, MountingHole:MountingHole_2.2mm_M2, symbol Mechanical:MountingHole
- F1: footprint Fuse:Fuse_1206_3216Metric -> Fuse:Fuse_0603_1608Metric
- J1: footprint Connector_USB:USB_C_Receptacle_GCT_USB4105-xx-A_16P_TopMnt_Horizontal -> Connector_USB:USB_C_Receptacle_HRO_TYPE-C-31-M-12
- J5: footprint Connector_PinSocket_2.54mm:PinSocket_1x06_P2.54mm_Horizontal -> Connector_PinSocket_2.54mm:PinSocket_1x06_P2.54mm_Vertical
Connections:
- net LROW4 is gone; now on net LRow 4: D16.1 (K), D31.1 (K), D8.1 (K)
- net LColumn 0: now also S8.1, U1.55 (PB3); no longer U1.28 (PB2)
- net LColumn 1: now also S16.1, U1.24 (PC4); no longer U1.53 (PC12)
- net LColumn 2: now also S31.1, U1.25 (PC5); no longer U1.55 (PB3)
- net LColumn 3: now also U1.51 (PC10); no longer U1.56 (PB4)
- net LColumn 4: now also U1.21 (PA5); no longer S8.1, U1.23 (PA7)
- net LColumn 5: now also U1.23 (PA7); no longer S16.1, U1.22 (PA6)
- net LColumn 6: now also U1.54 (PD2); no longer S31.1, U1.21 (PA5)
- net LRow 0: now also U1.53 (PC12); no longer U1.29 (PB10)
- net LRow 1: now also U1.56 (PB4); no longer U1.54 (PD2)
- net LRow 2: now also U1.22 (PA6); no longer U1.57 (PB5)
- net LRow 3: now also U1.52 (PC11); no longer U1.20 (PA4)
- net LTRACK_INT: no longer names the net of J4.4 (INT)
- net LTRACK_INT: no longer U1.51 (PC10)
- no-connect marks 21 -> 23
